File: Sprion-circuit/DRV8212.sch (KiCad schematic (older format))
At the start: 19 parts, among them U1 LM358, U2 LM358

Commit message: 電源でけたー！！
Connections:
- net labels added: +3.3VA
- net labels removed: VCC
Changed lines of the file:
@@
-$EndComp
-$Comp
-L power:VCC #PWR0106
-U 1 1 60EB4AD5
-P 1900 1700
-F 0 "#PWR0106" H 1900 1550 50  0001 C CNN
-F 1 "VCC" H 1915 1873 50  0000 C CNN
-F 2 "" H 1900 1700 50  0001 C CNN
-F 3 "" H 1900 1700 50  0001 C CNN
-	1    1900 1700
-	1    0    0    -1
 $EndComp
 $Comp
@@
 Text HLabel 3100 1950 0    50   Input ~ 0
 MD1_IN1
+$Comp
+L power:+3.3VA #PWR?
+U 1 1 60E5C849
+P 1900 1700
+F 0 "#PWR?" H 1900 1550 50  0001 C CNN
+F 1 "+3.3VA" H 1915 1873 50  0000 C CNN
+F 2 "" H 1900 1700 50  0001 C CNN
+F 3 "" H 1900 1700 50  0001 C CNN
+	1    1900 1700
+	1    0    0    -1
+$EndComp
 $EndSCHEMATC
