File: Sprion-circuit/Power.sch (KiCad schematic (older format))
At the start: 23 parts

Commit message: 電源でけたー！！
Parts:
- added C13: 10u, symbol Device:C
- added D1: LED, symbol Device:LED
- added L1: 47u, symbol Device:L
- added R17: R, symbol Device:R
- gave numbers to parts that had none: 23
Connections:
- net labels added: +3.3V, +3.3VA
- wire segments 57 -> 60
