File: Sprion-circuit/STM32f405.sch (KiCad schematic (older format))
At the start: 1 part

Commit message: 電源でけたー！！
Parts:
- gave numbers to parts that had none: 1
Changed lines of the file:
@@
 $EndDescr
 $Comp
-L MCU_ST_STM32F4:STM32F405RGTx U?
+L MCU_ST_STM32F4:STM32F405RGTx U3
 U 1 1 60F36A6E
 P 3300 3500
-F 0 "U?" H 3300 1611 50  0000 C CNN
+F 0 "U3" H 3300 1611 50  0000 C CNN
 F 1 "STM32F405RGTx" H 3300 1520 50  0000 C CNN
 F 2 "Package_QFP:LQFP-64_10x10mm_P0.5mm" H 2700 1800 50  0001 R CNN
