File: Sprion-circuit/Sprion-circuit.sch (KiCad schematic (older format))
At the start: 0 parts

Commit message: 電源でけたー！！
Changed lines of the file:
@@
 F0 "Power" 50
 F1 "Power.sch" 50
+F2 "BAT" I L 1300 3950 50
 $EndSheet
 $EndSCHEMATC
