File: Sprion-circuit/_autosave-Sprion-circuit.kicad_pcb (KiCad board)
At the start: 2 copper layers, 107.5 x 72 mm, 116 parts, among them IC1 R3111N211A, IC2 TAR5SB50, IC5 NJU6080F1, IC6 NJU6080F1, IC7 NJU6080F1, IC8 NJU6080F1, J1 Conn_01x03_Female, J2 Conn_01x04_Female, J3 Conn_02x03_Odd_Even, J4 Conn_02x03_Odd_Even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

Commit message: add,feat,fix:すまんコミットわすれててぐちゃぐちゃや
配置始めた。
フットプリント割り当てた
回路図pdfで吐いた
Parts:
- moved R24 173.7 mm to (174.7, 62.3), turned to 270 degrees
- moved C15 173.0 mm to (173.2, 65.3), turned to 270 degrees
- moved R25 170.4 mm to (174.7, 65.3), turned to 270 degrees
- moved C5 98.9 mm to (108.5, 90.3)
- moved RS2 97.0 mm to (108.6, 81.1)
- moved MD2 96.8 mm to (108.4, 88.3), turned to 180 degrees
- moved U5 90.3 mm to (108.9, 83.2), turned to 180 degrees
- moved RS1 84.5 mm to (108.7, 60.9)
- moved C2 78.3 mm to (108.8, 85.0)
- moved C1 73.4 mm to (108.8, 64.9)
- moved R32 69.0 mm to (167.1, 62.2), turned to 90 degrees
- moved U2 67.4 mm to (108.8, 63.0), turned to 180 degrees
- moved MD1 66.0 mm to (104.3, 60.8), turned to 180 degrees
- moved L1 62.9 mm to (170.2, 63.1)
- moved C4 59.4 mm to (102.1, 59.9), turned to 90 degrees
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