File: Sprion-circuit/IMU.sch (KiCad schematic (older format))
At the start: 5 parts

Commit message: fix: MD周り,タイマー割り当て
MDの書き方を変えた
タイマー割り当てを再構成、対称性・高性能タイマーをどうするかみたいなとこ
Connections:
- net IMU_INT: no longer names the net of U?.6 (INT)
- no-connect marks 0 -> 1
Changed lines of the file:
@@
 $Descr A4 11693 8268
 encoding utf-8
-Sheet 6 6
+Sheet 4 6
 Title ""
 Date ""
@@
 Wire Wire Line
 	6050 3000 5300 3000
-Text HLabel 5700 2900 2    50   Output ~ 0
-IMU_INT
-Wire Wire Line
-	5300 2900 5700 2900
 Text HLabel 4050 3100 0    50   BiDi ~ 0
 IMU_SPC
+NoConn ~ 5300 2900
 $EndSCHEMATC

Commit message: add,feat,fix:すまんコミットわすれててぐちゃぐちゃや
配置始めた。
フットプリント割り当てた
回路図pdfで吐いた
Parts:
- C36, C37, C38, C39: renamed from C?; footprint (none) -> Capacitor_SMD:C_0603_1608Metric
- gave numbers to parts that had none: 1
Connections:
- net +3V3: now also U1.1 (VDDIO), U1.16 (VDD)
- net GND: now also C36.2, C37.2, C38.2
Other:
- moved on the sheet: C36, C37, C38
Changed lines of the file:
@@
 $EndDescr
 $Comp
-L Sensor_Motion:ICM-20602 U?
+L Sensor_Motion:ICM-20602 U1
 U 1 1 61A9FA37
 P 4800 3000
-F 0 "U?" H 4800 2411 50  0000 C CNN
+F 0 "U1" H 4800 2411 50  0000 C CNN
 F 1 "ICM-20602" H 4800 2320 50  0000 C CNN
 F 2 "Package_LGA:LGA-16_3x3mm_P0.5mm_LayoutBorder3x5y" H 4800 3250 50  0001 C CNN
@@
 CS
 $Comp
-L power:GND #PWR?
+L power:GND #PWR090
 U 1 1 61AA4377
 P 4800 3500
-F 0 "#PWR?" H 4800 3250 50  0001 C CNN
+F 0 "#PWR090" H 4800 3250 50  0001 C CNN
 F 1 "GND" H 4805 3327 50  0000 C CNN
 F 2 "" H 4800 3500 50  0001 C CNN
@@
 $EndComp
 $Comp
-L power:+3.3V #PWR?
+L power:+3.3V #PWR089
 U 1 1 61AA6150
-P 4650 1750
-F 0 "#PWR?" H 4650 1600 50  0001 C CNN
-F 1 "+3.3V" H 4665 1923 50  0000 C CNN
-F 2 "" H 4650 1750 50  0001 C CNN
-F 3 "" H 4650 1750 50  0001 C CNN
-	1    4650 1750
+P 4650 2000
+F 0 "#PWR089" H 4650 1850 50  0001 C CNN
+F 1 "+3.3V" H 4665 2173 50  0000 C CNN
+F 2 "" H 4650 2000 50  0001 C CNN
+F 3 "" H 4650 2000 50  0001 C CNN
+	1    4650 2000
 	1    0    0    -1
 $EndComp
 $Comp
-L Device:C C?
+L Device:C C36
 U 1 1 61AA6FC5
-P 4200 1950
-F 0 "C?" H 4315 1996 50  0000 L CNN
-F 1 "0.1u" H 4315 1905 50  0000 L CNN
-F 2 "" H 4238 1800 50  0001 C CNN
-F 3 "~" H 4200 1950 50  0001 C CNN
-	1    4200 1950
+P 3550 2300
+F 0 "C36" H 3665 2346 50  0000 L CNN
+F 1 "0.1u" H 3665 2255 50  0000 L CNN
+F 2 "Capacitor_SMD:C_0603_1608Metric" H 3588 2150 50  0001 C CNN
+F 3 "~" H 3550 2300 50  0001 C CNN
+	1    3550 2300
 	1    0    0    -1
 $EndComp
 $Comp
-L Device:C C?
+L Device:C C37
 U 1 1 61AA7D2E
-P 4650 1950
-F 0 "C?" H 4765 1996 50  0000 L CNN
-F 1 "2.2u" H 4765 1905 50  0000 L CNN
-F 2 "" H 4688 1800 50  0001 C CNN
-F 3 "~" H 4650 1950 50  0001 C CNN
-	1    4650 1950
+P 4000 2300
+F 0 "C37" H 4115 2346 50  0000 L CNN
+F 1 "2.2u" H 4115 2255 50  0000 L CNN
+F 2 "Capacitor_SMD:C_0603_1608Metric" H 4038 2150 50  0001 C CNN
+F 3 "~" H 4000 2300 50  0001 C CNN
+	1    4000 2300
 	1    0    0    -1
 $EndComp
 $Comp
-L Device:C C?
+L Device:C C38
 U 1 1 61AA84C5
-P 5150 1950
-F 0 "C?" H 5265 1996 50  0000 L CNN
-F 1 "0.01u" H 5265 1905 50  0000 L CNN
-F 2 "" H 5188 1800 50  0001 C CNN
-F 3 "~" H 5150 1950 50  0001 C CNN
-	1    5150 1950
+P 5550 2300
+F 0 "C38" H 5665 2346 50  0000 L CNN
+F 1 "0.01u" H 5665 2255 50  0000 L CNN
+F 2 "Capacitor_SMD:C_0603_1608Metric" H 5588 2150 50  0001 C CNN
+F 3 "~" H 5550 2300 50  0001 C CNN
+	1    5550 2300
 	1    0    0    -1
 $EndComp
 $Comp
-L power:+3.3V #PWR?
+L power:+3.3V #PWR091
 U 1 1 61AB0193
-P 5150 1750
-F 0 "#PWR?" H 5150 1600 50  0001 C CNN
-F 1 "+3.3V" H 5165 1923 50  0000 C CNN
-F 2 "" H 5150 1750 50  0001 C CNN
-F 3 "" H 5150 1750 50  0001 C CNN
-	1    5150 1750
+P 5150 2000
+F 0 "#PWR091" H 5150 1850 50  0001 C CNN
+F 1 "+3.3V" H 5165 2173 50  0000 C CNN
+F 2 "" H 5150 2000 50  0001 C CNN
+F 3 "" H 5150 2000 50  0001 C CNN
+	1    5150 2000
 	1    0    0    -1
 $EndComp
 Wire Wire Line
-	4200 1800 4650 1800
-Wire Wire Line
-	4650 1750 4650 1800
-Connection ~ 4650 1800
-Wire Wire Line
-	5150 1750 5150 1800
-Wire Wire Line
-	4200 2100 4650 2100
-Wire Wire Line
-	4650 2100 4650 2500
-Wire Wire Line
 	4650 2500 4800 2500
-Connection ~ 4650 2100
 Wire Wire Line
 	4900 2500 5150 2500
-Wire Wire Line
-	5150 2500 5150 2100
 Wire Wire Line
 	4050 2900 4300 2900
@@
 	4300 3200 4050 3200
 $Comp
-L power:GND #PWR?
+L power:GND #PWR092
 U 1 1 61AB198D
 P 5700 3450
-F 0 "#PWR?" H 5700 3200 50  0001 C CNN
+F 0 "#PWR092" H 5700 3200 50  0001 C CNN
 F 1 "GND" H 5705 3277 50  0000 C CNN
 F 2 "" H 5700 3450 50  0001 C CNN
@@
 $EndComp
 $Comp
-L Device:C C?
+L Device:C C39
 U 1 1 61AB2A83
 P 5700 3250
-F 0 "C?" H 5815 3296 50  0000 L CNN
+F 0 "C39" H 5815 3296 50  0000 L CNN
 F 1 "0.1u" H 5815 3205 50  0000 L CNN
-F 2 "" H 5738 3100 50  0001 C CNN
+F 2 "Capacitor_SMD:C_0603_1608Metric" H 5738 3100 50  0001 C CNN
 F 3 "~" H 5700 3250 50  0001 C CNN
 	1    5700 3250
@@
 	5700 3400 5700 3450
 $Comp
-L power:GND #PWR?
+L power:GND #PWR093
 U 1 1 61AB43F5
 P 6050 3000
-F 0 "#PWR?" H 6050 2750 50  0001 C CNN
+F 0 "#PWR093" H 6050 2750 50  0001 C CNN
 F 1 "GND" H 6055 2827 50  0000 C CNN
 F 2 "" H 6050 3000 50  0001 C CNN
@@
 IMU_SPC
 NoConn ~ 5300 2900
+Wire Wire Line
+	4650 2000 4650 2150
+Wire Wire Line
+	4000 2150 4650 2150
+Connection ~ 4650 2150
+Wire Wire Line
+	4650 2150 4650 2500
+Wire Wire Line
+	3550 2150 4000 2150
+Connection ~ 4000 2150
+Wire Wire Line
+	3550 2450 3750 2450
+$Comp
+L power:GND #PWR098
+U 1 1 61B63C76
+P 3750 2450
+F 0 "#PWR098" H 3750 2200 50  0001 C CNN
+F 1 "GND" H 3755 2277 50  0000 C CNN
+F 2 "" H 3750 2450 50  0001 C CNN
+F 3 "" H 3750 2450 50  0001 C CNN
+	1    3750 2450
+	1    0    0    -1
+$EndComp
+Connection ~ 3750 2450
+Wire Wire Line
+	3750 2450 4000 2450
+Wire Wire Line
+	5150 2000 5150 2150
+Wire Wire Line
+	5550 2150 5150 2150
+Connection ~ 5150 2150
+Wire Wire Line
+	5150 2150 5150 2500
+$Comp
+L power:GND #PWR099
+U 1 1 61B67D0C
+P 5550 2450
+F 0 "#PWR099" H 5550 2200 50  0001 C CNN
+F 1 "GND" H 5555 2277 50  0000 C CNN
+F 2 "" H 5550 2450 50  0001 C CNN
+F 3 "" H 5550 2450 50  0001 C CNN
+	1    5550 2450
+	1    0    0    -1
+$EndComp
 $EndSCHEMATC
